Commit message: Add navigation from Nav2 package

File: simulation/ros2_sim_ws/src/robot_pkg/description/gazebo_control.xacro (robot description, xacro)
@@ -9,6 +9,4 @@
             <right_joint>right_back_wheel_joint</right_joint>
             <wheel_separation>0.36</wheel_separation>
-            <wheel_separation>0.36</wheel_separation>
-            <wheel_diameter>0.2</wheel_diameter>
             <wheel_diameter>0.2</wheel_diameter>
             <!-- Limits -->

File: simulation/ros2_sim_ws/src/robot_pkg/description/lidar.xacro (robot description, xacro)
@@ -4,5 +4,5 @@
         <parent link="chassis"/>
         <child link="laser_frame"/>
-        <origin xyz="0 0 0.1" rpy="0 0 0"/>
+        <origin xyz="0.3 0 0.17" rpy="0 0 0"/>
     </joint>
     <link name="laser_frame">

File: simulation/ros2_sim_ws/src/robot_pkg/description/robot_core.xacro (robot description, xacro)
@@ -1,4 +1,4 @@
 <?xml version="1.0"?>
-<robot xmlns:xacro="http://www.ros.org/wiki/xacro" >
+<robot name="diff_4_wheel" xmlns:xacro="http://www.ros.org/wiki/xacro" >
     <xacro:include filename="inertial_macros.xacro"/>
     <material name="white">
@@ -21,5 +21,5 @@
     <joint name="base_footprint_joint" type="fixed">
         <parent link="base_link"/>
-        <child link="base_footprint"/>
+            <child link="base_footprint"/>
         <origin xyz="0 0 0" rpy="0 0 0"/>
     </joint>
